File: PCB/Wemos-ESP32_MAX7219 v1.brd (EAGLE design)
At the start: 53 x 32.1 mm, 12 parts

Commit message: Minor corrections
Changed lines of the file:
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@@
 <contactref element="D11" pad="2"/>
 <contactref element="U$1" pad="11"/>
-<wire x1="9" y1="13.08" x2="8.2" y2="13.08" width="0.508" layer="16"/>
-<wire x1="8.2" y1="13.08" x2="7.4" y2="12.28" width="0.508" layer="16"/>
-<wire x1="18.8" y1="4.8" x2="20" y2="6" width="0.508" layer="16"/>
-<wire x1="7.4" y1="12.28" x2="7.4" y2="6.6" width="0.508" layer="16"/>
-<wire x1="7.4" y1="6.6" x2="9.2" y2="4.8" width="0.508" layer="16"/>
-<wire x1="9.2" y1="4.8" x2="18.8" y2="4.8" width="0.508" layer="16"/>
+<wire x1="9" y1="13.08" x2="8.2" y2="13.08" width="0.3048" layer="16"/>
+<wire x1="8.2" y1="13.08" x2="7.4" y2="12.28" width="0.3048" layer="16"/>
+<wire x1="18.8" y1="4.8" x2="20" y2="6" width="0.3048" layer="16"/>
+<wire x1="7.4" y1="12.28" x2="7.4" y2="6.6" width="0.3048" layer="16"/>
+<wire x1="7.4" y1="6.6" x2="9.2" y2="4.8" width="0.3048" layer="16"/>
+<wire x1="9.2" y1="4.8" x2="18.8" y2="4.8" width="0.3048" layer="16"/>
 </signal>
 <signal name="IO12">
 <contactref element="D12" pad="2"/>
 <contactref element="U$1" pad="12"/>
-<wire x1="9" y1="10.54" x2="10.3" y2="9.24" width="0.508" layer="1"/>
-<wire x1="10.3" y1="9.24" x2="10.3" y2="6.6" width="0.508" layer="1"/>
-<wire x1="10.3" y1="6.6" x2="12.1" y2="4.8" width="0.508" layer="1"/>
-<wire x1="23.1" y1="4.8" x2="24" y2="5.7" width="0.508" layer="1"/>
-<wire x1="24" y1="5.7" x2="24" y2="6" width="0.508" layer="1"/>
-<wire x1="12.1" y1="4.8" x2="23.1" y2="4.8" width="0.508" layer="1"/>
+<wire x1="9" y1="10.54" x2="10.3" y2="9.24" width="0.3048" layer="1"/>
+<wire x1="10.3" y1="9.24" x2="10.3" y2="6.6" width="0.3048" layer="1"/>
+<wire x1="10.3" y1="6.6" x2="12.1" y2="4.8" width="0.3048" layer="1"/>
+<wire x1="23.1" y1="4.8" x2="24" y2="5.7" width="0.3048" layer="1"/>
+<wire x1="24" y1="5.7" x2="24" y2="6" width="0.3048" layer="1"/>
+<wire x1="12.1" y1="4.8" x2="23.1" y2="4.8" width="0.3048" layer="1"/>
 </signal>
 </signals>
