File: PCB/Wemos-ESP8266_MAX7219 v5.sch (EAGLE design)
At the start: 11 parts

Commit message: Minor corrections
Other:
- note added: "Wemos D1 Mini - MAX7219 (c) Mats Karlsson 2023-05-29 v5"
- note removed: "Wemos D1 Mini - MAX7219 (c) Mats Karlsson 2023-04-24 v3"
Changed lines of the file:
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@@
 <wire x1="114.3" y1="60.96" x2="114.3" y2="0" width="0.6096" layer="98" style="longdash"/>
 <text x="2.794" y="2.286" size="1.778" layer="97">Wemos D1 Mini - MAX7219
-(c) Mats Karlsson 2023-04-24 v3</text>
+(c) Mats Karlsson 2023-05-29 v5</text>
 <text x="50.8" y="51.054" size="1.778" layer="97">D5 - CLK
 D6 - CS
